Commit message: fix pose panda_description

File: src/panda_description/urdf/arm.xacro (robot description, xacro)
@@ -3,4 +3,5 @@
   <!-- World Frame -->
   <link name="world"/>
+  <link name  ="tcp_link"/>
   <!-- Link 0 - Base -->
   <link name="panda_link0">
@@ -21,9 +22,9 @@
       </inertial>
   </link>
-  <!-- World-Base Joint -->
+  <!-- World-Base Joint  rpy="0 0 1.57 -->
   <joint name="virtual_joint" type="fixed">
     <parent link="world"/>
     <child link="panda_link0"/>
-    <origin xyz="0.6 0 0.35" rpy="0 0 1.57"/>
+    <origin xyz="0.6 0 0.35" rpy="0 0 0"/>
   </joint>
   <!-- Link 1 -->
@@ -180,12 +181,12 @@
       </inertial>
   </link>
-  <!-- Joint 6 -->
+  <!-- Joint 6 45 deg = 57079632679-->
   <joint name="panda_joint6" type="revolute">
-    <safety_controller k_position="100.0" k_velocity="40.0" soft_lower_limit="-0.0175" soft_upper_limit="3.7525"/>
-    <origin rpy="1.57079632679 0 0" xyz="0 0 0"/>
+    <safety_controller k_position="100.0" k_velocity="40.0" soft_lower_limit="-1.57079632679" soft_upper_limit="3.141562"/>
+    <origin rpy="1.57079632679 -1.57079632679 0 " xyz="0 0 0"/>
     <parent link="panda_link5"/>
     <child link="panda_link6"/>
     <axis xyz="0 0 1"/>
-    <limit effort="30.0" lower="-0.0873" upper="3.8223" velocity="10.0"/>
+    <limit effort="30.0" lower="-1.1873" upper="3.8223" velocity="10.0"/>
   </joint>
   <!-- Link 7 -->
@@ -216,4 +217,10 @@
     <limit effort="30.0" lower="-2.9671" upper="2.9671" velocity="10.0"/>
   </joint>
+  <!-- tcp_joint -->
+    <joint    name  ="tcp_joint"             type      ="fixed">
+    <origin xyz   ="0 0 0.08"              rpy       ="0 0 0"/>
+    <parent link  ="panda_hand"/>
+    <child  link  ="tcp_link"/>
+  </joint>
   <!-- Hand Link -->
   <link name="panda_hand">
@@ -234,5 +241,5 @@
       </inertial>
   </link>
-  <!-- Hand Joint -->
+  <!-- Hand Joint rpy="0 0 -0.785398163397 -->
   <joint name="panda_hand_joint" type="fixed">
     <parent link="panda_link7"/>

File: src/panda_description/urdf/ros2control.xacro (robot description, xacro)
@@ -2,19 +2,20 @@
 <robot xmlns:xacro="http://www.ros.org/wiki/xacro" name="panda">
   <xacro:property name="PI" value="3.14159265359" />
+  <xacro:arg name="use_mock_hardware" default="true" />
+  <xacro:arg name="is_ignition" default="false" />
   <ros2_control name="RobotSystem" type="system">
-    <!-- ros2_control Gazebo -->
-    <!-- ROS 2 Humble -->
-    <xacro:if value="$(arg is_ignition)">
-      <hardware>
-        <plugin>ign_ros2_control/IgnitionSystem</plugin>
-      </hardware>
-    </xacro:if>
-    <!-- ROS 2 Iron or above -->
-    <xacro:unless value="$(arg is_ignition)">
-      <hardware>
-        <plugin>gz_ros2_control/GazeboSimSystem</plugin>
-      </hardware>
-    </xacro:unless>
-    <!-- Joint 1 -->
+    <hardware>
+      <xacro:if value="$(arg use_mock_hardware)">
+        <plugin>mock_components/GenericSystem</plugin>
+      </xacro:if>
+      <xacro:unless value="$(arg use_mock_hardware)">
+        <xacro:if value="$(arg is_ignition)">
+          <plugin>ign_ros2_control/IgnitionSystem</plugin>
+        </xacro:if>
+        <xacro:unless value="$(arg is_ignition)">
+          <plugin>gz_ros2_control/GazeboSimSystem</plugin>
+        </xacro:unless>
+      </xacro:unless>
+    </hardware>
     <joint name="panda_joint1">
       <command_interface name="position">
@@ -24,5 +25,4 @@
       <state_interface name="position"/>
     </joint>
-    <!-- Joint 2 -->
     <joint name="panda_joint2">
       <command_interface name="position">
@@ -32,5 +32,4 @@
       <state_interface name="position"/>
     </joint>
-    <!-- Joint 3 -->
     <joint name="panda_joint3">
       <command_interface name="position">
@@ -40,5 +39,4 @@
       <state_interface name="position"/>
     </joint>
-    <!-- Joint 4 -->
     <joint name="panda_joint4">
       <command_interface name="position">
@@ -46,7 +44,8 @@
         <param name="max">0.0</param>
       </command_interface>
-      <state_interface name="position"/>
+      <state_interface name="position">
+        <param name="initial_value">-1.57</param>
+      </state_interface>
     </joint>
-    <!-- Joint 5 -->
     <joint name="panda_joint5">
       <command_interface name="position">
@@ -56,5 +55,4 @@
       <state_interface name="position"/>
     </joint>
-    <!-- Joint 6 -->
     <joint name="panda_joint6">
       <command_interface name="position">
@@ -64,5 +62,4 @@
       <state_interface name="position"/>
     </joint>
-    <!-- Joint 7 -->
     <joint name="panda_joint7">
       <command_interface name="position">
@@ -72,5 +69,4 @@
       <state_interface name="position"/>
     </joint>
-    <!-- Gripper Finger Joint 1 -->
     <joint name="panda_finger_joint1">
       <command_interface name="position">
@@ -80,5 +76,4 @@
       <state_interface name="position"/>
     </joint>
-    <!-- Gripper Finger Joint 2 (Mimics Joint 1) -->
     <joint name="panda_finger_joint2">
       <command_interface name="position">
