Commit message: update world + sensor astra

File: src/panda_description/urdf/panda.urdf.xacro (robot description, xacro)
@@ -6,3 +6,4 @@
   <xacro:include filename="$(find panda_description)/urdf/gazebo.xacro" />
   <xacro:include filename="$(find panda_description)/urdf/ros2control.xacro" />
+  <xacro:base_camera parent_link="panda_hand"/>
 </robot>

File: src/panda_description/urdf/sensors.xacro (robot description, xacro)
@@ -1,58 +1,86 @@
-<?xml version="1.0" ?>
-<robot name="panda" xmlns:xacro="http://www.ros.org/wiki/xacro">
-    <link name="camera_link">
+<?xml version="1.0"?>
+<robot xmlns:xacro="http://www.ros.org/wiki/xacro">
+    <xacro:macro name="base_camera"
+                params="parent_link
+                        base_link:=camera_link
+                        camera_name:=camera
+                        frame_name:=frame">
+      <link name="${base_link}">
         <inertial>
-            <origin xyz="0 0 0" rpy="0.0 0.0 0.0"/>
-            <mass value="0.1"/>
-            <inertia ixx="0.1" ixy="0.0" ixz="0.0" iyy="0.1" iyz="0.0" izz="0.1"/>
+          <origin xyz="0 0 0" rpy="0 0 0"/>
+          <mass value="0.1"/>
+          <inertia ixx="0.0001" ixy="0" ixz="0"
+                  iyy="0.0001" iyz="0"
+                  izz="0.0001"/>
         </inertial>
         <visual>
-            <origin xyz="0 0 0" rpy="0.0 0.0 0.0"/>
-            <geometry>
-                <box size="0.1 0.1 0.05"/>
-            </geometry>
-            <material name="red"/>
+          <origin xyz="0 0 0" rpy="0 0 0"/>
+          <geometry>
+            <mesh filename="package://panda_description/meshes/visual/astra_cam.stl"
+                  scale="1 1 1"/>
+          </geometry>
+          <material name="black">
+            <color rgba="0.05 0.05 0.05 1.0"/>
+          </material>
         </visual>
         <collision>
-            <origin xyz="0 0 0" rpy="0.0 0.0 0.0"/>
-            <geometry>
-                <box size="0.1 0.1 0.05"/>
-            </geometry>
-            <material name="red"/>
+          <origin xyz="0 0 0" rpy="0 0 0"/>
+          <geometry>
+            <box size="0.05 0.04 0.04"/>
+          </geometry>
         </collision>
-    </link>
-    <joint name="camera_joint" type="fixed">
-        <origin xyz="0.6 0 1.0" rpy="0.0 0.0 0.0"/>
-        <parent link="panda_link0"/>
-        <child link="camera_link"/>
-    </joint>
-    <link name="camera_link_optical" />
-    <joint name="camera_optical_joint" type="fixed">
-        <parent link="camera_link"/>
-        <child link="camera_link_optical"/>
+      </link>
+      <link name="${base_link}_optical"/>
+      <joint name="${base_link}_joint" type="fixed">
+        <parent link="${parent_link}"/>
+        <child link="${base_link}"/>
+        <origin xyz="0.05 0.0 0.06" rpy="0 0.785 0"/>
+      </joint>
+      <joint name="${base_link}_optical_joint" type="fixed">
+        <parent link="${base_link}"/>
+        <child link="${base_link}_optical"/>
         <origin xyz="0 0 0" rpy="${-pi/2} 0 ${-pi/2}"/>
-    </joint>
-    <gazebo reference="camera_link">
-        <sensor name="camera" type="camera">
-            <pose>0 0 0 0 1.57 0</pose>
-            <visualize>true</visualize>
-            <update_rate>10.0</update_rate>
-            <alwaysOn>true</alwaysOn>
-            <topic>camera/image_raw</topic>
-            <gz_frame_id>camera_link_optical</gz_frame_id>
-            <camera name="intel_realsense_r200">
-                <camera_info_topic>camera/camera_info</camera_info_topic>
-                <horizontal_fov>1.0</horizontal_fov>
-                <image>
-                    <width>640</width>
-                    <height>320</height>
-                    <format>R8G8B8</format>
-                </image>
-                <clip>
-                    <near>0.05</near>
-                    <far>8.0</far>
-                </clip>
-            </camera>
+      </joint>
+      <gazebo reference="${base_link}">
+        <sensor name="astra_rgb" type="camera">
+          <pose>0 0 0 0 0 0</pose>
+          <always_on>true</always_on>
+          <update_rate>30</update_rate>
+          <visualize>true</visualize>
+          <topic>/astra/rgb/image_raw</topic>
+          <gz_frame_id>${base_link}_optical</gz_frame_id>
+          <camera>
+            <image>
+              <width>640</width>
+              <height>480</height>
+              <format>R8G8B8</format>
+            </image>
+            <clip>
+              <near>0.05</near>
+              <far>8.0</far>
+            </clip>
+          </camera>
         </sensor>
-  </gazebo>
+      </gazebo>
+      <gazebo reference="${base_link}">
+        <sensor name="astra_depth" type="depth">
+          <pose>0 0 0 0 0 0</pose>
+          <always_on>true</always_on>
+          <update_rate>30</update_rate>
+          <visualize>true</visualize>
+          <topic>/astra/depth/image_raw</topic>
+          <gz_frame_id>${base_link}_optical</gz_frame_id>
+          <camera>
+            <image>
+              <width>640</width>
+              <height>480</height>
+            </image>
+            <clip>
+              <near>0.05</near>
+              <far>8.0</far>
+            </clip>
+          </camera>
+        </sensor>
+      </gazebo>
+    </xacro:macro>
 </robot>
